File: hardware/cpu_section.kicad_sch (KiCad schematic)
At the start: 49 parts, among them J1 Micro_SD_Card_Det1, J2 USB_B_Micro, J20 FTDI_PROGRAMMER, J21 ICSP, J37 LED_UI_CONNECTOR, Q11 BC547, SW2 ATMEL_RST, U1 W25Q32JVSS, U2 DS1307Z+, U3 74LVC125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

Commit message: ADDS production files
Parts:
- removed Q11: BC547, Package_TO_SOT_THT:TO-92_Inline, symbol Transistor_BJT:BC547
- added Q5: BC846, Package_TO_SOT_SMD:SOT-23, symbol Transistor_BJT:BC846
- U1: LCSC Part# (none) -> C82344
- U2: LCSC Part# (none) -> C9868
- U5: LCSC Part# (none) -> C22460
- Y2: LCSC Part# (none) -> C13738
Connections:
- net BUZZER: now also Q5.1 (B)
- net ESP_RX1: now also U5.13 (PH1); no longer U5.46 (PD3)
- net ESP_TX1: now also U5.12 (PH0); no longer U5.45 (PD2)
- net FLOW_METER_1: now also U5.25 (PB6); no longer U5.12 (PH0)
- net FLOW_METER_2: now also U5.26 (PB7); no longer U5.13 (PH1)
- net FLOW_METER_3: now also U5.45 (PD2); no longer U5.14 (PH2)
- net FLOW_METER_4: now also U5.46 (PD3); no longer U5.15 (PH3)
- net FLOW_METER_5: now also U5.6 (PE4); no longer U5.16 (PH4)
- net FLOW_METER_6: now also U5.7 (PE5); no longer U5.17 (PH5)
- net GND: now also Q5.2 (E)
- net at BZ1.2 (-): now also Q5.3 (C)
Other:
- moved on the sheet: C17, D4, J2, R15, R16
