File: hardware/master.kicad_sch (KiCad schematic)
At the start: 0 parts

Commit message: ADDS production files
Other:
- note added: "Hydros"
- note removed: "SMART IRRIGATION MANAGER"
Changed lines of the file:
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@@
 	(generator_version "9.0")
 	(paper "A4")
-	(text "SMART IRRIGATION MANAGER"
+	(text "Hydros"
 		(exclude_from_sim no)
-		(at 148.082 38.1 0)
+		(at 160.02 40.64 0)
 		(effects
 			(font
 				(size 8 8)
+				(thickness 1.6)
+				(bold yes)
 			)
 		)
