File: hardware/output_control.kicad_sch (KiCad schematic)
At the start: 61 parts, among them J27 REL1_TERMINAL, J28 REL2_TERMINAL, J29 REL3_TERMINAL, J30 REL4_TERMINAL, J31 REL5_TERMINAL, J32 REL6_TERMINAL, J33 REL7_TERMINAL, J34 REL8_TERMINAL, K1 SANYOU_SRD_Form_C, K2 SANYOU_SRD_Form_C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

Commit message: ADDS production files
Parts:
- K1, K2, K3, K4, K5: LCSC Part# (none) -> C35449
Changed lines of the file:
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@@
 	(text "FIXME: CHANGE TO AO3400\n"
 		(exclude_from_sim no)
-		(at 276.86 121.666 0)
+		(at 284.226 122.174 0)
 		(effects
 			(font
@@
 			)
 		)
+		(property "LCSC Part#" "C35449"
+			(at 153.67 113.03 0)
+			(effects
+				(font
+					(size 1.27 1.27)
+				)
+				(hide yes)
+			)
+		)
 		(pin "3"
 		)
@@
 			)
 		)
+		(property "LCSC Part#" "C35449"
+			(at 152.4 67.31 0)
+			(effects
+				(font
+					(size 1.27 1.27)
+				)
+				(hide yes)
+			)
+		)
 		(pin "3"
 		)
@@
 			)
 		)
+		(property "LCSC Part#" "C35449"
+			(at 153.67 156.21 0)
+			(effects
+				(font
+					(size 1.27 1.27)
+				)
+				(hide yes)
+			)
+		)
 		(pin "3"
 		)
@@
 			)
 		)
+		(property "LCSC Part#" "C35449"
+			(at 271.78 63.5 0)
+			(effects
+				(font
+					(size 1.27 1.27)
+				)
+				(hide yes)
+			)
+		)
 		(pin "3"
 		)
@@
 			(at 153.67 198.12 0)
 			(effects
+				(font
+					(size 1.27 1.27)
+				)
+				(hide yes)
+			)
+		)
+		(property "LCSC Part#" "C35449"
+			(at 153.67 198.12 0)
+			(effects
