File: hardware/power-supply-unit.kicad_sch (KiCad schematic)
At the start: 46 parts, among them J16 AC IN, J17 Jack-DC, J18 DC_EN, J19 AC_EN, Q9 Si4532DY, U15 TPS54308, U16 TPS62932, U17 TLV75533PDBV, U18 LTC4365TS8

Commit message: ADDS production files
Parts:
- added R66: 0R, Resistor_SMD:R_0805_2012Metric, symbol Device:R_Small
- D26: LCSC Part# (none) -> C86299
- PS1: LCSC Part# (none) -> C20616758
- Q9: LCSC Part# (none) -> C5123913; now not fitted; now left out of the parts list
- R46, R47, R48, R49, U18: now not fitted; now left out of the parts list
- R52: LCSC Part# (none) -> C2828857
- U15: LCSC Part# (none) -> C168839
- U16: LCSC Part# (none) -> C3032935
- U17: LCSC Part# (none) -> C404027
Connections:
- net 12V_DC: now also R66.1
- net at D26.1 (K), Q9.7 (D), Q9.8 (D)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: now also R66.2
Other:
- moved on the sheet: D26, J17
