File: hardware/sensors_and_inputs.kicad_sch (KiCad schematic)
At the start: 46 parts, among them J10 Flow Meter, J11 Flow Meter, J12 Flow Meter, J13 Flow Meter, J22 DS18B20_1, J23 DS18B20_2, J24 DS18B20_3, J25 DS18B20_4, J26 BH1750 LIGHT, J3 Flow Meter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

Commit message: ADDS production files
Parts:
- C21: LCSC Part# (none) -> C49678
- J7: LCSC Part# (none) -> C430601
- U13: LCSC Part# (none) -> C92489
- U6: LCSC Part# (none) -> C1549752
Changed lines of the file:
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@@
 			)
 		)
-		(property "LCSC Part#" ""
+		(property "LCSC Part#" "C49678"
 			(at 127 97.79 0)
 			(effects
@@
 			)
 		)
+		(property "LCSC Part#" "C1549752"
+			(at 285.75 120.65 0)
+			(effects
+				(font
+					(size 1.27 1.27)
+				)
+				(hide yes)
+			)
+		)
 		(pin "4"
 		)
@@
 			)
 		)
-		(property "LCSC Part#" ""
+		(property "LCSC Part#" "C430601"
 			(at 67.31 240.03 0)
 			(effects
@@
 			(at 190.5 179.07 0)
 			(effects
+				(font
+					(size 1.27 1.27)
+				)
+				(hide yes)
+			)
+		)
+		(property "LCSC Part#" "C92489"
+			(at 190.5 179.07 0)
+			(effects
