File: hardware/smart-irrigation-manager.kicad_pcb (KiCad board)
At the start: 2 copper layers, 209 x 124.7 mm, 202 parts, among them J1 Micro_SD_Card_Det1, J10 Flow Meter, J11 Flow Meter, J12 Flow Meter, J13 Flow Meter, J14 ESP-PROG, J15 BOOT-OPTION, J16 AC IN, J17 Jack-DC, J18 DC_EN, J19 AC_EN, J20 FTDI_PROGRAMMER, J21 ICSP, J22 DS18B20_1, J23 DS18B20_2, J24 DS18B20_3, J25 DS18B20_4, J26 BH1750 LIGHT, J27 REL1_TERMINAL, J28 REL2_TERMINAL, J29 REL3_TERMINAL, J3 Flow Meter, J30 REL4_TERMINAL, J31 REL5_TERMINAL, J35 20x4 LCD connector, J36 LED_UI_CONNECTOR, J37 LED_UI_CONNECTOR, J4 Soil Moisture Sensor 1, J5 Soil Moisture Sensor 2, J6 Soil Moisture Sensor 3, J7 Soil Moisture Sensor 5, J8 Soil Moisture Sensor 4, J9 Flow Meter, K1 SANYOU_SRD_Form_C, K2 SANYOU_SRD_Form_C, K3 SANYOU_SRD_Form_C, K4 SANYOU_SRD_Form_C, K5 SANYOU_SRD_Form_C, Q1 AO3400A, Q10 AO3400A, Q11 BC547, Q2 AO3400A, Q3 AO3400A, Q4 AO3400A, Q9 Si4532DY, SW1 RESET, SW2 ATMEL_RST, U1 W25Q32JVSS, U10 LM393, U11 LM393, U12 LM393, U13 BME280, U14 ESP32-S3-WROOM-1, U15 TPS54308, U16 TPS62932, U17 TLV75533PDBV, U18 LTC4365TS8, U2 DS1307Z+, U3 74LVC125, U4 TXB0104D, U5 ATmega2560-16A, U6 TXB0104D, U8 LM393, U9 LM393, Y1 32.768kHz, Y2 16MHz

Commit message: ADDS production files
Parts:
- removed Q11: BC547, Package_TO_SOT_THT:TO-92_Inline
- added G***: LOGO, my-footprints:spectrol-systems-logo-FCu, F.Cu at (112.9, -81.8)
- added Q5: BC846, Package_TO_SOT_SMD:SOT-23, F.Cu at (76.7, -129.3)
- added R66: 0R, Resistor_SMD:R_0805_2012Metric, F.Cu at (28.8, -179.4)
Connections:
- U5 pad 12: FLOW_METER_1 -> ESP_TX1
- U5 pad 13: FLOW_METER_2 -> ESP_RX1
- U5 pad 14: FLOW_METER_3 -> unconnected-(U5-PH2-Pad14)
- U5 pad 15: FLOW_METER_4 -> unconnected-(U5-PH3-Pad15)
- U5 pad 16: FLOW_METER_5 -> unconnected-(U5-PH4-Pad16)
- U5 pad 17: FLOW_METER_6 -> unconnected-(U5-PH5-Pad17)
- U5 pad 25: unconnected-(U5-PB6-Pad25) -> FLOW_METER_1
- U5 pad 26: unconnected-(U5-PB7-Pad26) -> FLOW_METER_2
- U5 pad 45: ESP_TX1 -> FLOW_METER_3
- U5 pad 46: ESP_RX1 -> FLOW_METER_4
- U5 pad 52: TEMP2 -> unconnected-(U5-PG1-Pad52)
- U5 pad 6: unconnected-(U5-PE4-Pad6) -> FLOW_METER_5
- U5 pad 7: unconnected-(U5-PE5-Pad7) -> FLOW_METER_6
- U5 pad 70: TEMP3 -> unconnected-(U5-PG2-Pad70)
- U5 pad 71: TEMP4 -> unconnected-(U5-PA7-Pad71)
Routing:
- net ESP_TX1: track 86.8 -> 60.5 mm
- net ESP_RX1: track 82.6 -> 59.3 mm
- net FLOW_METER_2: track 82.5 -> 105.6 mm
- net /Master/POWER SUPPLY UNIT/12V_DC: track 35.6 -> 55.7 mm, vias 0 -> 1
- net FLOW_METER_1: track 96.4 -> 76.8 mm
- net FLOW_METER_4: track 111.6 -> 128.5 mm, vias 3 -> 7
- net Net-(D26-K): track 82.2 -> 96.1 mm, vias 0 -> 2
- net FLOW_METER_3: track 98.8 -> 102.0 mm, vias 3 -> 6
- net SD_DETECT: track 77.5 -> 80.5 mm
- net /Master/CPU_SECTION/BUZZER: track 14.1 -> 16.6 mm
- net Net-(BZ1--): track 10.8 -> 12.4 mm
- net FLOW_METER_6: track 130.1 -> 130.8 mm
- net (no net): vias 2 -> 0
