File: hardware/userinterface.kicad_sch (KiCad schematic)
At the start: 12 parts, among them J35 20x4 LCD connector, J36 LED_UI_CONNECTOR

Commit message: ADDS production files
Changed lines of the file:
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@@
 	(text "LED INDICATION STRIP TO BE MOUNTED OFF-BOARD\nAND CONNECTED TO MOTHERBOARD USING JST CONNECTOR\nAS LABELLED\n"
 		(exclude_from_sim no)
-		(at 199.136 98.806 0)
+		(at 202.184 98.806 0)
 		(effects
 			(font
