File: hardware/wifi_and_comms.kicad_sch (KiCad schematic)
At the start: 14 parts, among them J14 ESP-PROG, J15 BOOT-OPTION, SW1 RESET, U14 ESP32-S3-WROOM-1

Commit message: ADDS production files
Parts:
- U14: LCSC Part# (none) -> C2913198
Changed lines of the file:
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@@
+			)
+		)
+		(property "LCSC Part#" "C2913198"
+			(at 236.22 149.86 0)
+			(effects
+				(font
+					(size 1.27 1.27)
+				)
+				(hide yes)
 			)
 		)
